File: sdrac_board/MCU.kicad_sch (KiCad schematic)
At the start: 36 parts, among them J1 SWD, J11 SYNCHRONIZER, SW1 BOOT0, SW2 NRST, SW3 USR_BTN, U1 FM24CL16B, U2 STM32F412RGT6, Y1 16MHz

Commit message: fixed caps and added nreset
Parts:
- removed J1: SWD, Connector_PinHeader_2.54mm:PinHeader_1x03_P2.54mm_Vertical, symbol Connector_Generic:Conn_01x03
- added C14: 2.2u, Capacitor_SMD:C_0603_1608Metric, symbol Device:C
- added J12: SWD, Connector_PinHeader_2.54mm:PinHeader_1x04_P2.54mm_Vertical, symbol Connector_Generic:Conn_01x04
Connections:
- net GND: now also C14.2, J12.1 (Pin_1)
- net NRST: now also J12.4 (Pin_4)
- net SWCLK: now also J12.2 (Pin_2)
- net SWDIO: now also J12.3 (Pin_3)
- net at U2.30 (VCAP_1): now also C14.1
- no-connect marks 24 -> 23
Changed lines of the file:
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@@
   (no_connect (at 167.64 124.46))
   (no_connect (at 132.08 81.28))
-  (no_connect (at 132.08 121.92))
   (no_connect (at 167.64 104.14))
   (no_connect (at 167.64 73.66))
@@
     (stroke (width 0) (type default))
   )
-  (wire (pts (xy 254 38.1) (xy 255.27 38.1))
-    (stroke (width 0) (type default))
-  )
   (wire (pts (xy 191.77 35.56) (xy 200.66 35.56))
     (stroke (width 0) (type default))
@@
     (stroke (width 0) (type default))
   )
+  (wire (pts (xy 125.73 121.92) (xy 132.08 121.92))
+    (stroke (width 0) (type default))
+  )
   (wire (pts (xy 185.42 35.56) (xy 191.77 35.56))
     (stroke (width 0) (type default))
@@
     (stroke (width 0) (type default))
   )
-  (polyline (pts (xy 270.51 26.67) (xy 270.51 46.99))
+  (polyline (pts (xy 269.24 26.67) (xy 269.24 44.45))
     (stroke (width 0) (type default))
   )
@@
     (stroke (width 0) (type default))
   )
+  (wire (pts (xy 251.46 38.1) (xy 251.46 40.64))
+    (stroke (width 0) (type default))
+  )
   (wire (pts (xy 96.52 73.66) (xy 96.52 71.12))
     (stroke (width 0) (type default))
@@
     (stroke (width 0) (type default))
   )
-  (polyline (pts (xy 240.03 46.99) (xy 240.03 26.67))
+  (polyline (pts (xy 238.76 44.45) (xy 238.76 26.67))
     (stroke (width 0) (type default))
   )
@@
     (stroke (width 0) (type default))
   )
+  (wire (pts (xy 125.73 124.46) (xy 125.73 121.92))
+    (stroke (width 0) (type default))
+  )
   (wire (pts (xy 129.54 99.06) (xy 132.08 99.06))
     (stroke (width 0) (type default))
@@
     (stroke (width 0) (type default))
   )
-  (wire (pts (xy 254 35.56) (xy 255.27 35.56))
-    (stroke (width 0) (type default))
-  )
   (wire (pts (xy 27.94 132.08) (xy 27.94 133.35))
     (stroke (width 0) (type default))
@@
     (stroke (width 0) (type default))
   )
-  (wire (pts (xy 254 40.64) (xy 254 41.91))
-    (stroke (width 0) (type default))
-  )
   (wire (pts (xy 172.72 35.56) (xy 172.72 36.83))
     (stroke (width 0) (type default))
   )
-  (wire (pts (xy 255.27 40.64) (xy 254 40.64))
-    (stroke (width 0) (type default))
-  )
   (wire (pts (xy 167.64 114.3) (xy 170.18 114.3))
     (stroke (width 0) (type default))
@@
     (stroke (width 0) (type default))
   )
+  (wire (pts (xy 252.73 30.48) (xy 256.54 30.48))
+    (stroke (width 0) (type default))
+  )
   (wire (pts (xy 144.78 35.56) (xy 147.32 35.56))
     (stroke (width 0) (type default))
@@
     (stroke (width 0) (type default))
   )
+  (wire (pts (xy 125.73 133.35) (xy 125.73 132.08))
+    (stroke (width 0) (type default))
+  )
   (wire (pts (xy 152.4 50.8) (xy 152.4 49.53))
     (stroke (width 0) (type default))
@@
     (stroke (width 0) (type default))
   )
-  (polyline (pts (xy 240.03 26.67) (xy 270.51 26.67))
+  (polyline (pts (xy 238.76 26.67) (xy 269.24 26.67))
     (stroke (width 0) (type default))
   )
@@
     (stroke (width 0) (type default))
   )
+  (wire (pts (xy 252.73 33.02) (xy 256.54 33.02))
+    (stroke (width 0) (type default))
+  )
   (wire (pts (xy 191.77 44.45) (xy 191.77 45.72))
     (stroke (width 0) (type default))
@@
     (stroke (width 0) (type default))
   )
-  (polyline (pts (xy 240.03 46.99) (xy 270.51 46.99))
+  (polyline (pts (xy 238.76 44.45) (xy 269.24 44.45))
     (stroke (width 0) (type default))
   )
@@
     (stroke (width 0) (type default))
   )
+  (wire (pts (xy 256.54 38.1) (xy 251.46 38.1))
+    (stroke (width 0) (type default))
+  )
   (wire (pts (xy 167.64 86.36) (xy 171.45 86.36))
     (stroke (width 0) (type default))
@@
   )
   (wire (pts (xy 209.55 34.29) (xy 209.55 35.56))
+    (stroke (width 0) (type default))
+  )
+  (wire (pts (xy 252.73 35.56) (xy 256.54 35.56))
     (stroke (width 0) (type default))
   )
@@
     (effects (font (size 1.27 1.27)) (justify left bottom))
   )
-  (text "SWD" (at 241.3 31.75 0)
+  (text "SWD" (at 241.3 40.64 0)
     (effects (font (size 2.54 2.54)) (justify left bottom))
   )
@@
     (effects (font (size 1.27 1.27)) (justify right bottom))
   )
-  (label "SWDIO" (at 254 35.56 180) (fields_autoplaced)
+  (label "SWDIO" (at 252.73 33.02 180) (fields_autoplaced)
     (effects (font (size 1.27 1.27)) (justify right bottom))
   )
@@
     (effects (font (size 1.27 1.27)) (justify left bottom))
   )
+  (label "NRST" (at 252.73 30.48 180) (fields_autoplaced)
+    (effects (font (size 1.27 1.27)) (justify right bottom))
+  )
   (label "USR_LED2" (at 129.54 96.52 180) (fields_autoplaced)
     (effects (font (size 1.27 1.27)) (justify right bottom))
@@
     (effects (font (size 1.27 1.27)) (justify right bottom))
   )
-  (label "SWCLK" (at 254 38.1 180) (fields_autoplaced)
+  (label "SWCLK" (at 252.73 35.56 180) (fields_autoplaced)
     (effects (font (size 1.27 1.27)) (justify right bottom))
   )
@@
     (effects (font (size 1.27 1.27)) (justify left))
   )
+  (symbol (lib_id "Device:C") (at 125.73 128.27 0) (unit 1)
+    (in_bom yes) (on_board yes) (dnp no)
+    (property "Reference" "C14" (at 127 125.73 0)
+      (effects (font (size 1.27 1.27)) (justify left))
+    )
+    (property "Value" "2.2u" (at 127 130.81 0)
+      (effects (font (size 1.27 1.27)) (justify left))
+    )
+    (property "Footprint" "Capacitor_SMD:C_0603_1608Metric" (at 126.6952 132.08 0)
+      (effects (font (size 1.27 1.27)) hide)
+    )
+    (property "Datasheet" "~" (at 125.73 128.27 0)
+      (effects (font (size 1.27 1.27)) hide)
+    )
+    (pin "1")
+    (pin "2")
+    (instances
+      (project "sdrac_board"
+        (path "/7e6d1db5-12f1-49d6-b3bd-d624ec5345e8/bf443dee-dc39-4dae-8f50-a44c6afacc04"
+          (reference "C14") (unit 1)
+        )
+      )
+    )
+  )
   (symbol (lib_id "Device:C") (at 153.67 40.64 0) (unit 1)
     (in_bom yes) (on_board yes) (dnp no)
@@
     )
   )
-  (symbol (lib_id "power:GND") (at 254 41.91 0) (unit 1)
-    (in_bom yes) (on_board yes) (dnp no)
-    (property "Reference" "#PWR022" (at 254 48.26 0)
-      (effects (font (size 1.27 1.27)) hide)
-    )
-    (property "Value" "GND" (at 254 45.72 0)
-      (effects (font (size 1.27 1.27)) hide)
-    )
-    (property "Footprint" "" (at 254 41.91 0)
-      (effects (font (size 1.27 1.27)) hide)
-    )
-    (property "Datasheet" "" (at 254 41.91 0)
+  (symbol (lib_id "power:GND") (at 251.46 40.64 0) (unit 1)
+    (in_bom yes) (on_board yes) (dnp no)
+    (property "Reference" "#PWR022" (at 251.46 46.99 0)
+      (effects (font (size 1.27 1.27)) hide)
+    )
+    (property "Value" "GND" (at 251.46 44.45 0)
+      (effects (font (size 1.27 1.27)) hide)
+    )
+    (property "Footprint" "" (at 251.46 40.64 0)
+      (effects (font (size 1.27 1.27)) hide)
+    )
+    (property "Datasheet" "" (at 251.46 40.64 0)
       (effects (font (size 1.27 1.27)) hide)
     )
@@
         (path "/98359aeb-e3f0-4579-a083-8ca5fb10d8d7/22fd861a-846b-4d74-8793-40be3c328ac6"
           (reference "#PWR014") (unit 1)
+        )
+      )
+    )
+  )
+  (symbol (lib_id "Connector_Generic:Conn_01x04") (at 261.62 35.56 0) (mirror x) (unit 1)
+    (in_bom yes) (on_board yes) (dnp no)
+    (property "Reference" "J12" (at 264.16 35.56 0)
+      (effects (font (size 1.27 1.27)) (justify left))
+    )
+    (property "Value" "SWD" (at 264.16 33.02 0)
+      (effects (font (size 1.27 1.27)) (justify left))
+    )
+    (property "Footprint" "Connector_PinHeader_2.54mm:PinHeader_1x04_P2.54mm_Vertical" (at 261.62 35.56 0)
+      (effects (font (size 1.27 1.27)) hide)
+    )
+    (property "Datasheet" "~" (at 261.62 35.56 0)
+      (effects (font (size 1.27 1.27)) hide)
+    )
+    (pin "2")
+    (pin "4")
+    (pin "3")
+    (pin "1")
+    (instances
+      (project "sdrac_board"
+        (path "/7e6d1db5-12f1-49d6-b3bd-d624ec5345e8/bf443dee-dc39-4dae-8f50-a44c6afacc04"
+          (reference "J12") (unit 1)
         )
       )
@@
     )
   )
-  (symbol (lib_id "Connector_Generic:Conn_01x03") (at 260.35 38.1 0) (unit 1)
-    (in_bom yes) (on_board yes) (dnp no) (fields_autoplaced)
-    (property "Reference" "J1" (at 262.89 36.8299 0)
-      (effects (font (size 1.27 1.27)) (justify left))
-    )
-    (property "Value" "SWD" (at 262.89 39.3699 0)
-      (effects (font (size 1.27 1.27)) (justify left))
-    )
-    (property "Footprint" "Connector_PinHeader_2.54mm:PinHeader_1x03_P2.54mm_Vertical" (at 260.35 38.1 0)
-      (effects (font (size 1.27 1.27)) hide)
-    )
-    (property "Datasheet" "~" (at 260.35 38.1 0)
-      (effects (font (size 1.27 1.27)) hide)
-    )
-    (pin "1")
-    (pin "2")
-    (pin "3")
-    (instances
-      (project "sdrac_board"
-        (path "/7e6d1db5-12f1-49d6-b3bd-d624ec5345e8/bf443dee-dc39-4dae-8f50-a44c6afacc04"
-          (reference "J1") (unit 1)
-        )
-      )
-      (project "motor controller"
-        (path "/98359aeb-e3f0-4579-a083-8ca5fb10d8d7/22fd861a-846b-4d74-8793-40be3c328ac6"
-          (reference "J2") (unit 1)
-        )
-      )
-    )
-  )
   (symbol (lib_id "Device:Crystal_GND24") (at 96.52 67.31 90) (unit 1)
     (in_bom yes) (on_board yes) (dnp no)
@@
         )
       )
+    )
+  )
+  (symbol (lib_name "GND_1") (lib_id "power:GND") (at 125.73 133.35 0) (unit 1)
+    (in_bom yes) (on_board yes) (dnp no) (fields_autoplaced)
+    (property "Reference" "#PWR088" (at 125.73 139.7 0)
+      (effects (font (size 1.27 1.27)) hide)
+    )
+    (property "Value" "GND" (at 125.73 138.43 0)
+      (effects (font (size 1.27 1.27)) hide)
+    )
+    (property "Footprint" "" (at 125.73 133.35 0)
+      (effects (font (size 1.27 1.27)) hide)
+    )
+    (property "Datasheet" "" (at 125.73 133.35 0)
+      (effects (font (size 1.27 1.27)) hide)
+    )
+    (pin "1")
+    (instances
+      (project "sdrac_board"
+        (path "/7e6d1db5-12f1-49d6-b3bd-d624ec5345e8/bf443dee-dc39-4dae-8f50-a44c6afacc04"
+          (reference "#PWR088") (unit 1)
+        )
+      )

Commit message: addded 6pin conenctor
Parts:
- added J1: INOUT, Connector_PinHeader_2.54mm:PinHeader_1x06_P2.54mm_Vertical, symbol Connector_Generic:Conn_01x06
Connections:
- net GND: now also J1.1 (Pin_1)
- net C_A1: now reaches U2.21 (PA5)
- net C_A1: now also J1.5 (Pin_5)
- net C_A2: now reaches U2.23 (PA7)
- net C_A2: now also J1.4 (Pin_4)
- net C_D1: now reaches U2.24 (PC4)
- net C_D1: now also J1.3 (Pin_3)
- net C_D2: now reaches U2.25 (PC5)
- net C_D2: now also J1.2 (Pin_2)
- new net +5V: J1.6 (Pin_6)
- no-connect marks 23 -> 19
Changed lines of the file:
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@@
   (no_connect (at 132.08 81.28))
   (no_connect (at 167.64 104.14))
-  (no_connect (at 167.64 73.66))
   (no_connect (at 132.08 109.22))
-  (no_connect (at 167.64 68.58))
-  (no_connect (at 132.08 88.9))
-  (no_connect (at 132.08 91.44))
   (no_connect (at 132.08 114.3))
   (no_connect (at 167.64 134.62))
@@
     (stroke (width 0) (type default))
   )
+  (wire (pts (xy 254 109.22) (xy 252.73 109.22))
+    (stroke (width 0) (type default))
+  )
   (wire (pts (xy 179.07 35.56) (xy 185.42 35.56))
     (stroke (width 0) (type default))
@@
     (stroke (width 0) (type default))
   )
+  (wire (pts (xy 252.73 109.22) (xy 252.73 111.76))
+    (stroke (width 0) (type default))
+  )
   (wire (pts (xy 129.54 96.52) (xy 132.08 96.52))
     (stroke (width 0) (type default))
@@
     (stroke (width 0) (type default))
   )
+  (wire (pts (xy 129.54 88.9) (xy 132.08 88.9))
+    (stroke (width 0) (type default))
+  )
   (wire (pts (xy 154.94 49.53) (xy 152.4 49.53))
     (stroke (width 0) (type default))
@@
     (stroke (width 0) (type default))
   )
+  (wire (pts (xy 129.54 91.44) (xy 132.08 91.44))
+    (stroke (width 0) (type default))
+  )
   (wire (pts (xy 147.32 35.56) (xy 153.67 35.56))
     (stroke (width 0) (type default))
@@
     (stroke (width 0) (type default))
   )
+  (wire (pts (xy 250.19 104.14) (xy 254 104.14))
+    (stroke (width 0) (type default))
+  )
   (wire (pts (xy 129.54 93.98) (xy 132.08 93.98))
     (stroke (width 0) (type default))
@@
     (stroke (width 0) (type default))
   )
+  (wire (pts (xy 250.19 99.06) (xy 254 99.06))
+    (stroke (width 0) (type default))
+  )
   (wire (pts (xy 149.86 142.24) (xy 149.86 143.51))
     (stroke (width 0) (type default))
@@
     (stroke (width 0) (type default))
   )
+  (wire (pts (xy 254 96.52) (xy 251.46 96.52))
+    (stroke (width 0) (type default))
+  )
   (wire (pts (xy 167.64 88.9) (xy 170.18 88.9))
     (stroke (width 0) (type default))
@@
     (stroke (width 0) (type default))
   )
+  (wire (pts (xy 167.64 73.66) (xy 170.18 73.66))
+    (stroke (width 0) (type default))
+  )
   (wire (pts (xy 172.72 35.56) (xy 172.72 36.83))
     (stroke (width 0) (type default))
   )
+  (wire (pts (xy 251.46 96.52) (xy 251.46 93.98))
+    (stroke (width 0) (type default))
+  )
   (wire (pts (xy 167.64 114.3) (xy 170.18 114.3))
     (stroke (width 0) (type default))
@@
     (stroke (width 0) (type default))
   )
+  (wire (pts (xy 167.64 68.58) (xy 170.18 68.58))
+    (stroke (width 0) (type default))
+  )
   (wire (pts (xy 49.53 167.64) (xy 49.53 168.91))
     (stroke (width 0) (type default))
@@
     (stroke (width 0) (type default))
   )
+  (wire (pts (xy 250.19 106.68) (xy 254 106.68))
+    (stroke (width 0) (type default))
+  )
   (wire (pts (xy 35.56 133.35) (xy 43.18 133.35))
+    (stroke (width 0) (type default))
+  )
+  (wire (pts (xy 250.19 101.6) (xy 254 101.6))
     (stroke (width 0) (type default))
   )
@@
     (effects (font (size 1.27 1.27)) (justify right bottom))
   )
+  (label "C_D2" (at 250.19 106.68 180) (fields_autoplaced)
+    (effects (font (size 1.27 1.27)) (justify right bottom))
+  )
   (label "3V3_MCU" (at 190.5 35.56 0) (fields_autoplaced)
     (effects (font (size 1.27 1.27)) (justify left bottom))
@@
     (effects (font (size 1.27 1.27)) (justify right bottom))
   )
+  (label "C_A1" (at 250.19 99.06 180) (fields_autoplaced)
+    (effects (font (size 1.27 1.27)) (justify right bottom))
+  )
+  (label "C_D2" (at 129.54 91.44 180) (fields_autoplaced)
+    (effects (font (size 1.27 1.27)) (justify right bottom))
+  )
   (label "OSC_OUT" (at 114.3 68.58 0) (fields_autoplaced)
     (effects (font (size 1.27 1.27)) (justify left bottom))
   )
+  (label "C_D1" (at 250.19 104.14 180) (fields_autoplaced)
+    (effects (font (size 1.27 1.27)) (justify right bottom))
+  )
   (label "USR_LED1" (at 129.54 93.98 180) (fields_autoplaced)
     (effects (font (size 1.27 1.27)) (justify right bottom))
@@
     (effects (font (size 1.27 1.27)) (justify left bottom))
   )
+  (label "C_A1" (at 170.18 68.58 0) (fields_autoplaced)
+    (effects (font (size 1.27 1.27)) (justify left bottom))
+  )
   (label "NRST" (at 252.73 30.48 180) (fields_autoplaced)
     (effects (font (size 1.27 1.27)) (justify right bottom))
@@
     (effects (font (size 1.27 1.27)) (justify right bottom))
   )
+  (label "C_D1" (at 129.54 88.9 180) (fields_autoplaced)
+    (effects (font (size 1.27 1.27)) (justify right bottom))
+  )
+  (label "C_A2" (at 250.19 101.6 180) (fields_autoplaced)
+    (effects (font (size 1.27 1.27)) (justify right bottom))
+  )
   (label "DIR_SYNC" (at 231.14 81.28 180) (fields_autoplaced)
     (effects (font (size 1.27 1.27)) (justify right bottom))
@@
   (label "SWCLK" (at 252.73 35.56 180) (fields_autoplaced)
     (effects (font (size 1.27 1.27)) (justify right bottom))
+  )
+  (label "C_A2" (at 170.18 73.66 0) (fields_autoplaced)
+    (effects (font (size 1.27 1.27)) (justify left bottom))
   )
   (label "USR_LED2" (at 48.26 167.64 180) (fields_autoplaced)
@@
         (path "/98359aeb-e3f0-4579-a083-8ca5fb10d8d7/22fd861a-846b-4d74-8793-40be3c328ac6"
           (reference "R10") (unit 1)
+        )
+      )
+    )
+  )
+  (symbol (lib_id "Connector_Generic:Conn_01x06") (at 259.08 104.14 0) (mirror x) (unit 1)
+    (in_bom yes) (on_board yes) (dnp no)
+    (property "Reference" "J1" (at 261.62 104.14 0)
+      (effects (font (size 1.27 1.27)) (justify left))
+    )
+    (property "Value" "INOUT" (at 261.62 101.6 0)
+      (effects (font (size 1.27 1.27)) (justify left))
+    )
+    (property "Footprint" "Connector_PinHeader_2.54mm:PinHeader_1x06_P2.54mm_Vertical" (at 259.08 104.14 0)
+      (effects (font (size 1.27 1.27)) hide)
+    )
+    (property "Datasheet" "~" (at 259.08 104.14 0)
+      (effects (font (size 1.27 1.27)) hide)
+    )
+    (pin "2")
+    (pin "1")
+    (pin "4")
+    (pin "3")
+    (pin "6")
+    (pin "5")
+    (instances
+      (project "sdrac_board"
+        (path "/7e6d1db5-12f1-49d6-b3bd-d624ec5345e8/bf443dee-dc39-4dae-8f50-a44c6afacc04"
+          (reference "J1") (unit 1)
         )
       )
@@
     )
   )
+  (symbol (lib_id "power:GND") (at 252.73 111.76 0) (unit 1)
+    (in_bom yes) (on_board yes) (dnp no)
+    (property "Reference" "#PWR089" (at 252.73 118.11 0)
+      (effects (font (size 1.27 1.27)) hide)
+    )
+    (property "Value" "GND" (at 252.73 115.57 0)
+      (effects (font (size 1.27 1.27)) hide)
+    )
+    (property "Footprint" "" (at 252.73 111.76 0)
+      (effects (font (size 1.27 1.27)) hide)
+    )
+    (property "Datasheet" "" (at 252.73 111.76 0)
+      (effects (font (size 1.27 1.27)) hide)
+    )
+    (pin "1")
+    (instances
+      (project "sdrac_board"
+        (path "/7e6d1db5-12f1-49d6-b3bd-d624ec5345e8/bf443dee-dc39-4dae-8f50-a44c6afacc04"
+          (reference "#PWR089") (unit 1)
+        )
+      )
+    )
+  )
   (symbol (lib_id "Device:C") (at 88.9 60.96 90) (unit 1)
     (in_bom yes) (on_board yes) (dnp no)
@@
         )
       )
+    )
+  )
+  (symbol (lib_id "power:+5V") (at 251.46 93.98 0) (unit 1)
+    (in_bom yes) (on_board yes) (dnp no) (fields_autoplaced)
+    (property "Reference" "#PWR090" (at 251.46 97.79 0)
+      (effects (font (size 1.27 1.27)) hide)
+    )
+    (property "Value" "+5V" (at 251.46 88.9 0)
+      (effects (font (size 1.27 1.27)))
+    )
+    (property "Footprint" "" (at 251.46 93.98 0)
+      (effects (font (size 1.27 1.27)) hide)
+    )
+    (property "Datasheet" "" (at 251.46 93.98 0)
+      (effects (font (size 1.27 1.27)) hide)
+    )
+    (pin "1")
+    (instances
+      (project "sdrac_board"
+        (path "/7e6d1db5-12f1-49d6-b3bd-d624ec5345e8/bf443dee-dc39-4dae-8f50-a44c6afacc04"
+          (reference "#PWR090") (unit 1)
+        )
+      )

Commit message: updated stuf
Other:
- note added: "ADC1 in1"
- note added: "ADC1 in14"
- note added: "ADC1 in15"
- note added: "ADC1 in2"
- note added: "ADC1 in3"
- note added: "ADC1 in4"
- note added: "Boards synchronization"
- note added: "Boot Reset"
- note added: "I2C"
- note added: "In Out Conector"
- note added: "Timer14 CH1 / ADC1 in7"
- note added: "Timer8 Ch1/ ADC1 in5"
- note removed: "Wejścia ANALOG"
- moved on the sheet: C1, C47, J1, J11, J12, R10, R34, R35, R4, R6, R9, SW1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

Commit message: stuff
Parts:
- J1: footprint Connector_PinHeader_2.54mm:PinHeader_1x06_P2.54mm_Vertical -> Connector_JST:JST_XH_B6B-XH-A_1x06_P2.50mm_Vertical
- J11: footprint Connector_PinHeader_2.54mm:PinHeader_1x02_P2.54mm_Vertical -> Connector_JST:JST_XH_B2B-XH-A_1x02_P2.50mm_Vertical
Changed lines of the file:
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@@
       (effects (font (size 1.27 1.27)) (justify left))
     )
-    (property "Footprint" "Connector_PinHeader_2.54mm:PinHeader_1x02_P2.54mm_Vertical" (at 259.08 44.45 0)
+    (property "Footprint" "Connector_JST:JST_XH_B2B-XH-A_1x02_P2.50mm_Vertical" (at 259.08 44.45 0)
       (effects (font (size 1.27 1.27)) hide)
     )
@@
       (effects (font (size 1.27 1.27)) (justify left))
     )
-    (property "Footprint" "Connector_PinHeader_2.54mm:PinHeader_1x06_P2.54mm_Vertical" (at 266.7 77.47 0)
-      (effects (font (size 1.27 1.27)) hide)
-    )
+    (property "Footprint" "Connector_JST:JST_XH_B6B-XH-A_1x06_P2.50mm_Vertical" (at 266.7 77.47 0)
+      (effects (font (size 1.27 1.27)) hide)
+    )

Commit message: made critical changes
Connections:
- net C_TX: now reaches U2.29 (PB10)
- net C_TX: now also J1.2 (Pin_2)
- net C_D1 renamed C_RX
- net C_D2: no longer names the net of U2.25 (PC5)
- net C_D2: no longer J1.2 (Pin_2)
Other:
- note added: "ADC1 in14/ UART3 RX"
- note added: "UART3 TX"
- note removed: "ADC1 in14"
- note removed: "ADC1 in15"
Changed lines of the file:
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@@
   )
   (no_connect (at 132.08 86.36))
-  (no_connect (at 167.64 124.46))
   (no_connect (at 132.08 81.28))
+  (no_connect (at 132.08 91.44))
   (no_connect (at 167.64 104.14))
   (no_connect (at 132.08 109.22))
@@
     (stroke (width 0) (type default))
   )
-  (wire (pts (xy 129.54 91.44) (xy 132.08 91.44))
-    (stroke (width 0) (type default))
-  )
   (wire (pts (xy 147.32 35.56) (xy 153.67 35.56))
     (stroke (width 0) (type default))
@@
     (stroke (width 0) (type default))
   )
+  (wire (pts (xy 170.18 124.46) (xy 167.64 124.46))
+    (stroke (width 0) (type default))
+  )
   (wire (pts (xy 147.32 44.45) (xy 147.32 45.72))
     (stroke (width 0) (type default))
@@
     (fill (type none))
   )
-  (text "ADC1 in15" (at 114.3 91.44 0)
-    (effects (font (size 1.27 1.27)) (justify left bottom))
+  (text "UART3 TX" (at 186.69 124.46 0)
+    (effects (font (size 1.27 1.27)) (justify right bottom))
   )
   (text "FRAM" (at 19.05 105.41 0)
@@
     (effects (font (size 1.27 1.27)) (justify left bottom))
   )
-  (text "ADC1 in14" (at 114.3 88.9 0)
+  (text "ADC1 in14/ UART3 RX" (at 102.87 88.9 0)
     (effects (font (size 1.27 1.27)) (justify left bottom))
   )
@@
     (effects (font (size 1.27 1.27)) (justify right bottom))
   )
-  (label "C_D2" (at 257.81 80.01 180) (fields_autoplaced)
+  (label "C_TX" (at 257.81 80.01 180) (fields_autoplaced)
     (effects (font (size 1.27 1.27)) (justify right bottom))
   )
@@
     (effects (font (size 1.27 1.27)) (justify right bottom))
   )
-  (label "C_D2" (at 129.54 91.44 180) (fields_autoplaced)
-    (effects (font (size 1.27 1.27)) (justify right bottom))
+  (label "C_TX" (at 170.18 124.46 0) (fields_autoplaced)
+    (effects (font (size 1.27 1.27)) (justify left bottom))
   )
   (label "OSC_OUT" (at 114.3 68.58 0) (fields_autoplaced)
     (effects (font (size 1.27 1.27)) (justify left bottom))
   )
-  (label "C_D1" (at 257.81 77.47 180) (fields_autoplaced)
+  (label "C_RX" (at 257.81 77.47 180) (fields_autoplaced)
     (effects (font (size 1.27 1.27)) (justify right bottom))
   )
@@
     (effects (font (size 1.27 1.27)) (justify right bottom))
   )
-  (label "C_D1" (at 129.54 88.9 180) (fields_autoplaced)
-    (effects (font (size 1.27 1.27)) (justify right bottom))
-  )
+  (label "C_RX" (at 129.54 88.9 180) (fields_autoplaced)
+    (effects (font (size 1.27 1.27)) (justify right bottom))
+  )
