File: sdrac_board/CAN.kicad_sch (KiCad schematic)
At the start: 10 parts, among them SW4 SW_DIP_x01, U3 SN65HVD232, U4 CAN, U5 CAN

Commit message: added second I2C communscation lane for synchronization and added wyas to change mcirosteping with resistors
Parts:
- renumbered C11 to C14, R14 to R16, R12 to R17, R13 to R18
Changed lines of the file:
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@@
   (symbol (lib_id "Device:R") (at 81.28 90.17 0) (unit 1)
     (in_bom yes) (on_board yes) (dnp no)
-    (property "Reference" "R12" (at 82.55 88.9 0)
+    (property "Reference" "R17" (at 82.55 88.9 0)
       (effects (font (size 1.27 1.27)) (justify left))
     )
@@
       (project "sdrac_board"
         (path "/7e6d1db5-12f1-49d6-b3bd-d624ec5345e8/8d618019-369d-4b89-bfb3-81126d20c35a"
-          (reference "R12") (unit 1)
+          (reference "R17") (unit 1)
         )
       )
@@
   (symbol (lib_id "power:GND") (at 106.68 104.14 0) (unit 1)
     (in_bom yes) (on_board yes) (dnp no)
-    (property "Reference" "#PWR024" (at 106.68 110.49 0)
+    (property "Reference" "#PWR031" (at 106.68 110.49 0)
       (effects (font (size 1.27 1.27)) hide)
     )
@@
       (project "sdrac_board"
         (path "/7e6d1db5-12f1-49d6-b3bd-d624ec5345e8/8d618019-369d-4b89-bfb3-81126d20c35a"
-          (reference "#PWR024") (unit 1)
+          (reference "#PWR031") (unit 1)
         )
       )
@@
   (symbol (lib_id "power:GND") (at 81.28 104.14 0) (unit 1)
     (in_bom yes) (on_board yes) (dnp no)
-    (property "Reference" "#PWR023" (at 81.28 110.49 0)
+    (property "Reference" "#PWR030" (at 81.28 110.49 0)
       (effects (font (size 1.27 1.27)) hide)
     )
@@
       (project "sdrac_board"
         (path "/7e6d1db5-12f1-49d6-b3bd-d624ec5345e8/8d618019-369d-4b89-bfb3-81126d20c35a"
-          (reference "#PWR023") (unit 1)
+          (reference "#PWR030") (unit 1)
         )
       )
@@
   (symbol (lib_id "Device:C") (at 135.89 92.71 0) (unit 1)
     (in_bom yes) (on_board yes) (dnp no)
-    (property "Reference" "C11" (at 137.16 90.17 0)
+    (property "Reference" "C14" (at 137.16 90.17 0)
       (effects (font (size 1.27 1.27)) (justify left))
     )
@@
       (project "sdrac_board"
         (path "/7e6d1db5-12f1-49d6-b3bd-d624ec5345e8/8d618019-369d-4b89-bfb3-81126d20c35a"
+          (reference "C14") (unit 1)
+        )
+      )
+      (project "motor controller"
+        (path "/98359aeb-e3f0-4579-a083-8ca5fb10d8d7/18447c1b-abaa-46e9-8bd6-d5f0c204f642"
           (reference "C11") (unit 1)
         )
       )
-      (project "motor controller"
-        (path "/98359aeb-e3f0-4579-a083-8ca5fb10d8d7/18447c1b-abaa-46e9-8bd6-d5f0c204f642"
-          (reference "C11") (unit 1)
-        )
-      )
     )
   )
   (symbol (lib_id "Device:R") (at 106.68 90.17 0) (unit 1)
     (in_bom yes) (on_board yes) (dnp no)
-    (property "Reference" "R13" (at 107.95 88.9 0)
+    (property "Reference" "R18" (at 107.95 88.9 0)
       (effects (font (size 1.27 1.27)) (justify left))
     )
@@
       (project "sdrac_board"
         (path "/7e6d1db5-12f1-49d6-b3bd-d624ec5345e8/8d618019-369d-4b89-bfb3-81126d20c35a"
-          (reference "R13") (unit 1)
+          (reference "R18") (unit 1)
         )
       )
@@
   (symbol (lib_id "power:+3V3") (at 135.89 81.28 0) (unit 1)
     (in_bom yes) (on_board yes) (dnp no)
-    (property "Reference" "#PWR025" (at 135.89 85.09 0)
+    (property "Reference" "#PWR028" (at 135.89 85.09 0)
       (effects (font (size 1.27 1.27)) hide)
     )
@@
       (project "sdrac_board"
         (path "/7e6d1db5-12f1-49d6-b3bd-d624ec5345e8/8d618019-369d-4b89-bfb3-81126d20c35a"
-          (reference "#PWR025") (unit 1)
+          (reference "#PWR028") (unit 1)
         )
       )
@@
   (symbol (lib_id "power:+3V3") (at 171.45 83.82 0) (unit 1)
     (in_bom yes) (on_board yes) (dnp no)
-    (property "Reference" "#PWR027" (at 171.45 87.63 0)
+    (property "Reference" "#PWR029" (at 171.45 87.63 0)
       (effects (font (size 1.27 1.27)) hide)
     )
@@
       (project "sdrac_board"
         (path "/7e6d1db5-12f1-49d6-b3bd-d624ec5345e8/8d618019-369d-4b89-bfb3-81126d20c35a"
-          (reference "#PWR027") (unit 1)
+          (reference "#PWR029") (unit 1)
         )
       )
@@
   (symbol (lib_id "Device:R") (at 207.01 74.93 90) (unit 1)
     (in_bom yes) (on_board yes) (dnp no)
-    (property "Reference" "R14" (at 207.01 72.39 90)
+    (property "Reference" "R16" (at 207.01 72.39 90)
       (effects (font (size 1.27 1.27)))
     )
@@
       (project "sdrac_board"
         (path "/7e6d1db5-12f1-49d6-b3bd-d624ec5345e8/8d618019-369d-4b89-bfb3-81126d20c35a"
-          (reference "R14") (unit 1)
+          (reference "R16") (unit 1)
         )
       )
@@
   (symbol (lib_id "power:GND") (at 171.45 104.14 0) (unit 1)
     (in_bom yes) (on_board yes) (dnp no)
-    (property "Reference" "#PWR028" (at 171.45 110.49 0)
+    (property "Reference" "#PWR033" (at 171.45 110.49 0)
       (effects (font (size 1.27 1.27)) hide)
     )
@@
       (project "sdrac_board"
         (path "/7e6d1db5-12f1-49d6-b3bd-d624ec5345e8/8d618019-369d-4b89-bfb3-81126d20c35a"
-          (reference "#PWR028") (unit 1)
+          (reference "#PWR033") (unit 1)
         )
       )
@@
   (symbol (lib_id "power:GND") (at 201.93 104.14 0) (unit 1)
     (in_bom yes) (on_board yes) (dnp no)
-    (property "Reference" "#PWR029" (at 201.93 110.49 0)
+    (property "Reference" "#PWR034" (at 201.93 110.49 0)
       (effects (font (size 1.27 1.27)) hide)
     )
@@
       (project "sdrac_board"
         (path "/7e6d1db5-12f1-49d6-b3bd-d624ec5345e8/8d618019-369d-4b89-bfb3-81126d20c35a"
-          (reference "#PWR029") (unit 1)
+          (reference "#PWR034") (unit 1)
         )
       )
@@
   (symbol (lib_id "power:GND") (at 222.25 104.14 0) (unit 1)
     (in_bom yes) (on_board yes) (dnp no)
-    (property "Reference" "#PWR030" (at 222.25 110.49 0)
+    (property "Reference" "#PWR035" (at 222.25 110.49 0)
       (effects (font (size 1.27 1.27)) hide)
     )
@@
       (project "sdrac_board"
         (path "/7e6d1db5-12f1-49d6-b3bd-d624ec5345e8/8d618019-369d-4b89-bfb3-81126d20c35a"
-          (reference "#PWR030") (unit 1)
+          (reference "#PWR035") (unit 1)
         )
       )
@@
   (symbol (lib_id "power:GND") (at 135.89 104.14 0) (unit 1)
     (in_bom yes) (on_board yes) (dnp no)
-    (property "Reference" "#PWR026" (at 135.89 110.49 0)
+    (property "Reference" "#PWR032" (at 135.89 110.49 0)
       (effects (font (size 1.27 1.27)) hide)
     )
@@
       (project "sdrac_board"
         (path "/7e6d1db5-12f1-49d6-b3bd-d624ec5345e8/8d618019-369d-4b89-bfb3-81126d20c35a"
-          (reference "#PWR026") (unit 1)
-        )
-      )
+          (reference "#PWR032") (unit 1)
+        )
+      )

Commit message: added hardware address selector
Parts:
- renumbered R16 to R22, R17 to R23, R18 to R24
Changed lines of the file:
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@@
   (symbol (lib_id "Device:R") (at 81.28 90.17 0) (unit 1)
     (in_bom yes) (on_board yes) (dnp no)
-    (property "Reference" "R17" (at 82.55 88.9 0)
+    (property "Reference" "R23" (at 82.55 88.9 0)
       (effects (font (size 1.27 1.27)) (justify left))
     )
@@
       (project "sdrac_board"
         (path "/7e6d1db5-12f1-49d6-b3bd-d624ec5345e8/8d618019-369d-4b89-bfb3-81126d20c35a"
-          (reference "R17") (unit 1)
+          (reference "R23") (unit 1)
         )
       )
@@
   (symbol (lib_id "power:GND") (at 106.68 104.14 0) (unit 1)
     (in_bom yes) (on_board yes) (dnp no)
-    (property "Reference" "#PWR031" (at 106.68 110.49 0)
+    (property "Reference" "#PWR037" (at 106.68 110.49 0)
       (effects (font (size 1.27 1.27)) hide)
     )
@@
       (project "sdrac_board"
         (path "/7e6d1db5-12f1-49d6-b3bd-d624ec5345e8/8d618019-369d-4b89-bfb3-81126d20c35a"
-          (reference "#PWR031") (unit 1)
+          (reference "#PWR037") (unit 1)
         )
       )
@@
   (symbol (lib_id "power:GND") (at 81.28 104.14 0) (unit 1)
     (in_bom yes) (on_board yes) (dnp no)
-    (property "Reference" "#PWR030" (at 81.28 110.49 0)
+    (property "Reference" "#PWR036" (at 81.28 110.49 0)
       (effects (font (size 1.27 1.27)) hide)
     )
@@
       (project "sdrac_board"
         (path "/7e6d1db5-12f1-49d6-b3bd-d624ec5345e8/8d618019-369d-4b89-bfb3-81126d20c35a"
-          (reference "#PWR030") (unit 1)
+          (reference "#PWR036") (unit 1)
         )
       )
@@
   (symbol (lib_id "Device:R") (at 106.68 90.17 0) (unit 1)
     (in_bom yes) (on_board yes) (dnp no)
-    (property "Reference" "R18" (at 107.95 88.9 0)
+    (property "Reference" "R24" (at 107.95 88.9 0)
       (effects (font (size 1.27 1.27)) (justify left))
     )
@@
       (project "sdrac_board"
         (path "/7e6d1db5-12f1-49d6-b3bd-d624ec5345e8/8d618019-369d-4b89-bfb3-81126d20c35a"
-          (reference "R18") (unit 1)
+          (reference "R24") (unit 1)
         )
       )
@@
   (symbol (lib_id "power:+3V3") (at 135.89 81.28 0) (unit 1)
     (in_bom yes) (on_board yes) (dnp no)
-    (property "Reference" "#PWR028" (at 135.89 85.09 0)
+    (property "Reference" "#PWR034" (at 135.89 85.09 0)
       (effects (font (size 1.27 1.27)) hide)
     )
@@
       (project "sdrac_board"
         (path "/7e6d1db5-12f1-49d6-b3bd-d624ec5345e8/8d618019-369d-4b89-bfb3-81126d20c35a"
-          (reference "#PWR028") (unit 1)
+          (reference "#PWR034") (unit 1)
         )
       )
@@
   (symbol (lib_id "power:+3V3") (at 171.45 83.82 0) (unit 1)
     (in_bom yes) (on_board yes) (dnp no)
-    (property "Reference" "#PWR029" (at 171.45 87.63 0)
+    (property "Reference" "#PWR035" (at 171.45 87.63 0)
       (effects (font (size 1.27 1.27)) hide)
     )
@@
       (project "sdrac_board"
         (path "/7e6d1db5-12f1-49d6-b3bd-d624ec5345e8/8d618019-369d-4b89-bfb3-81126d20c35a"
-          (reference "#PWR029") (unit 1)
+          (reference "#PWR035") (unit 1)
         )
       )
@@
   (symbol (lib_id "Device:R") (at 207.01 74.93 90) (unit 1)
     (in_bom yes) (on_board yes) (dnp no)
-    (property "Reference" "R16" (at 207.01 72.39 90)
+    (property "Reference" "R22" (at 207.01 72.39 90)
       (effects (font (size 1.27 1.27)))
     )
@@
       (project "sdrac_board"
         (path "/7e6d1db5-12f1-49d6-b3bd-d624ec5345e8/8d618019-369d-4b89-bfb3-81126d20c35a"
-          (reference "R16") (unit 1)
+          (reference "R22") (unit 1)
         )
       )
@@
   (symbol (lib_id "power:GND") (at 171.45 104.14 0) (unit 1)
     (in_bom yes) (on_board yes) (dnp no)
-    (property "Reference" "#PWR033" (at 171.45 110.49 0)
+    (property "Reference" "#PWR039" (at 171.45 110.49 0)
       (effects (font (size 1.27 1.27)) hide)
     )
@@
       (project "sdrac_board"
         (path "/7e6d1db5-12f1-49d6-b3bd-d624ec5345e8/8d618019-369d-4b89-bfb3-81126d20c35a"
+          (reference "#PWR039") (unit 1)
+        )
+      )
+      (project "motor controller"
+        (path "/98359aeb-e3f0-4579-a083-8ca5fb10d8d7/18447c1b-abaa-46e9-8bd6-d5f0c204f642"
+          (reference "#PWR032") (unit 1)
+        )
+      )
+    )
+  )
+  (symbol (lib_id "power:GND") (at 201.93 104.14 0) (unit 1)
+    (in_bom yes) (on_board yes) (dnp no)
+    (property "Reference" "#PWR040" (at 201.93 110.49 0)
+      (effects (font (size 1.27 1.27)) hide)
+    )
+    (property "Value" "GND" (at 201.93 107.95 0)
+      (effects (font (size 1.27 1.27)) hide)
+    )
+    (property "Footprint" "" (at 201.93 104.14 0)
+      (effects (font (size 1.27 1.27)) hide)
+    )
+    (property "Datasheet" "" (at 201.93 104.14 0)
+      (effects (font (size 1.27 1.27)) hide)
+    )
+    (pin "1")
+    (instances
+      (project "sdrac_board"
+        (path "/7e6d1db5-12f1-49d6-b3bd-d624ec5345e8/8d618019-369d-4b89-bfb3-81126d20c35a"
+          (reference "#PWR040") (unit 1)
+        )
+      )
+      (project "motor controller"
+        (path "/98359aeb-e3f0-4579-a083-8ca5fb10d8d7/18447c1b-abaa-46e9-8bd6-d5f0c204f642"
           (reference "#PWR033") (unit 1)
         )
       )
-      (project "motor controller"
-        (path "/98359aeb-e3f0-4579-a083-8ca5fb10d8d7/18447c1b-abaa-46e9-8bd6-d5f0c204f642"
-          (reference "#PWR032") (unit 1)
-        )
-      )
-    )
-  )
-  (symbol (lib_id "power:GND") (at 201.93 104.14 0) (unit 1)
-    (in_bom yes) (on_board yes) (dnp no)
-    (property "Reference" "#PWR034" (at 201.93 110.49 0)
-      (effects (font (size 1.27 1.27)) hide)
-    )
-    (property "Value" "GND" (at 201.93 107.95 0)
-      (effects (font (size 1.27 1.27)) hide)
-    )
-    (property "Footprint" "" (at 201.93 104.14 0)
-      (effects (font (size 1.27 1.27)) hide)
-    )
-    (property "Datasheet" "" (at 201.93 104.14 0)
-      (effects (font (size 1.27 1.27)) hide)
-    )
-    (pin "1")
-    (instances
-      (project "sdrac_board"
-        (path "/7e6d1db5-12f1-49d6-b3bd-d624ec5345e8/8d618019-369d-4b89-bfb3-81126d20c35a"
-          (reference "#PWR034") (unit 1)
-        )
-      )
-      (project "motor controller"
-        (path "/98359aeb-e3f0-4579-a083-8ca5fb10d8d7/18447c1b-abaa-46e9-8bd6-d5f0c204f642"
-          (reference "#PWR033") (unit 1)
-        )
-      )
     )
   )
   (symbol (lib_id "power:GND") (at 222.25 104.14 0) (unit 1)
     (in_bom yes) (on_board yes) (dnp no)
-    (property "Reference" "#PWR035" (at 222.25 110.49 0)
+    (property "Reference" "#PWR041" (at 222.25 110.49 0)
       (effects (font (size 1.27 1.27)) hide)
     )
@@
       (project "sdrac_board"
         (path "/7e6d1db5-12f1-49d6-b3bd-d624ec5345e8/8d618019-369d-4b89-bfb3-81126d20c35a"
-          (reference "#PWR035") (unit 1)
+          (reference "#PWR041") (unit 1)
         )
       )
@@
   (symbol (lib_id "power:GND") (at 135.89 104.14 0) (unit 1)
     (in_bom yes) (on_board yes) (dnp no)
-    (property "Reference" "#PWR032" (at 135.89 110.49 0)
+    (property "Reference" "#PWR038" (at 135.89 110.49 0)
       (effects (font (size 1.27 1.27)) hide)
     )
@@
       (project "sdrac_board"
         (path "/7e6d1db5-12f1-49d6-b3bd-d624ec5345e8/8d618019-369d-4b89-bfb3-81126d20c35a"
-          (reference "#PWR032") (unit 1)
-        )
-      )
+          (reference "#PWR038") (unit 1)
+        )
+      )

Commit message: added 10A screw terminal
Parts:
- SW4: footprint Button_Switch_SMD:SW_DIP_SPSTx01_Slide_6.7x4.1mm_W8.61mm_P2.54mm_LowProfile -> Button_Switch_SMD:SW_DIP_SPSTx01_Slide_6.7x4.1mm_W6.73mm_P2.54mm_LowProfile_JPin
Changed lines of the file:
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@@
       (effects (font (size 1.27 1.27)))
     )
-    (property "Footprint" "Button_Switch_SMD:SW_DIP_SPSTx01_Slide_6.7x4.1mm_W8.61mm_P2.54mm_LowProfile" (at 219.71 74.93 0)
+    (property "Footprint" "Button_Switch_SMD:SW_DIP_SPSTx01_Slide_6.7x4.1mm_W6.73mm_P2.54mm_LowProfile_JPin" (at 219.71 74.93 0)
       (effects (font (size 1.27 1.27)) hide)
     )
