File: sdrac_board/Sensors.kicad_sch (KiCad schematic)
At the start: 9 parts, among them J10 Pos_zero_sens, J7 Conn_01x02, J8 Conn_01x02, J9 Mag_enc, U11 MCP9700AT-ETT

Commit message: added second I2C communscation lane for synchronization and added wyas to change mcirosteping with resistors
Parts:
- renumbered C43 to C49, J9 to J10, J10 to J11, J8 to J12, J7 to J9, R31 to R41, R33 to R42, R32 to R43

Commit message: added hardware address selector
Parts:
- renumbered R41 to R47, R42 to R48, R43 to R49
Changed lines of the file:
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@@
   (symbol (lib_id "power:GND") (at 125.73 93.98 0) (unit 1)
     (in_bom yes) (on_board yes) (dnp no)
-    (property "Reference" "#PWR093" (at 125.73 100.33 0)
+    (property "Reference" "#PWR099" (at 125.73 100.33 0)
       (effects (font (size 1.27 1.27)) hide)
     )
@@
       (project "sdrac_board"
         (path "/7e6d1db5-12f1-49d6-b3bd-d624ec5345e8/0c32a19a-a7ea-4fd5-9033-ebbe7320ca24"
-          (reference "#PWR093") (unit 1)
+          (reference "#PWR099") (unit 1)
         )
       )
@@
   (symbol (lib_id "power:+5V") (at 181.61 74.93 0) (unit 1)
     (in_bom yes) (on_board yes) (dnp no)
-    (property "Reference" "#PWR090" (at 181.61 78.74 0)
+    (property "Reference" "#PWR096" (at 181.61 78.74 0)
       (effects (font (size 1.27 1.27)) hide)
     )
@@
       (project "sdrac_board"
         (path "/7e6d1db5-12f1-49d6-b3bd-d624ec5345e8/0c32a19a-a7ea-4fd5-9033-ebbe7320ca24"
-          (reference "#PWR090") (unit 1)
+          (reference "#PWR096") (unit 1)
         )
       )
@@
   (symbol (lib_id "power:+3V3") (at 82.55 95.25 0) (unit 1)
     (in_bom yes) (on_board yes) (dnp no)
-    (property "Reference" "#PWR094" (at 82.55 99.06 0)
+    (property "Reference" "#PWR0100" (at 82.55 99.06 0)
       (effects (font (size 1.27 1.27)) hide)
     )
@@
       (project "sdrac_board"
         (path "/7e6d1db5-12f1-49d6-b3bd-d624ec5345e8/0c32a19a-a7ea-4fd5-9033-ebbe7320ca24"
-          (reference "#PWR094") (unit 1)
+          (reference "#PWR0100") (unit 1)
         )
       )
@@
   (symbol (lib_id "power:GND") (at 82.55 81.28 0) (unit 1)
     (in_bom yes) (on_board yes) (dnp no)
-    (property "Reference" "#PWR091" (at 82.55 87.63 0)
+    (property "Reference" "#PWR097" (at 82.55 87.63 0)
       (effects (font (size 1.27 1.27)) hide)
     )
@@
       (project "sdrac_board"
         (path "/7e6d1db5-12f1-49d6-b3bd-d624ec5345e8/0c32a19a-a7ea-4fd5-9033-ebbe7320ca24"
-          (reference "#PWR091") (unit 1)
+          (reference "#PWR097") (unit 1)
         )
       )
@@
   (symbol (lib_id "power:GND") (at 82.55 107.95 0) (unit 1)
     (in_bom yes) (on_board yes) (dnp no)
-    (property "Reference" "#PWR098" (at 82.55 114.3 0)
+    (property "Reference" "#PWR0104" (at 82.55 114.3 0)
       (effects (font (size 1.27 1.27)) hide)
     )
@@
       (project "sdrac_board"
         (path "/7e6d1db5-12f1-49d6-b3bd-d624ec5345e8/0c32a19a-a7ea-4fd5-9033-ebbe7320ca24"
-          (reference "#PWR098") (unit 1)
+          (reference "#PWR0104") (unit 1)
         )
       )
@@
   (symbol (lib_id "power:+3V3") (at 82.55 69.85 0) (unit 1)
     (in_bom yes) (on_board yes) (dnp no)
-    (property "Reference" "#PWR087" (at 82.55 73.66 0)
+    (property "Reference" "#PWR093" (at 82.55 73.66 0)
       (effects (font (size 1.27 1.27)) hide)
     )
@@
       (project "sdrac_board"
         (path "/7e6d1db5-12f1-49d6-b3bd-d624ec5345e8/0c32a19a-a7ea-4fd5-9033-ebbe7320ca24"
-          (reference "#PWR087") (unit 1)
+          (reference "#PWR093") (unit 1)
         )
       )
@@
   (symbol (lib_id "power:GND") (at 185.42 104.14 270) (unit 1)
     (in_bom yes) (on_board yes) (dnp no)
-    (property "Reference" "#PWR097" (at 179.07 104.14 0)
+    (property "Reference" "#PWR0103" (at 179.07 104.14 0)
       (effects (font (size 1.27 1.27)) hide)
     )
@@
       (project "sdrac_board"
         (path "/7e6d1db5-12f1-49d6-b3bd-d624ec5345e8/0c32a19a-a7ea-4fd5-9033-ebbe7320ca24"
-          (reference "#PWR097") (unit 1)
+          (reference "#PWR0103") (unit 1)
         )
       )
@@
   (symbol (lib_id "power:+3V3") (at 175.26 74.93 0) (unit 1)
     (in_bom yes) (on_board yes) (dnp no)
-    (property "Reference" "#PWR089" (at 175.26 78.74 0)
+    (property "Reference" "#PWR095" (at 175.26 78.74 0)
       (effects (font (size 1.27 1.27)) hide)
     )
@@
       (project "sdrac_board"
         (path "/7e6d1db5-12f1-49d6-b3bd-d624ec5345e8/0c32a19a-a7ea-4fd5-9033-ebbe7320ca24"
-          (reference "#PWR089") (unit 1)
+          (reference "#PWR095") (unit 1)
         )
       )
@@
   (symbol (lib_id "power:+3V3") (at 177.8 97.79 0) (unit 1)
     (in_bom yes) (on_board yes) (dnp no)
-    (property "Reference" "#PWR095" (at 177.8 101.6 0)
+    (property "Reference" "#PWR0101" (at 177.8 101.6 0)
       (effects (font (size 1.27 1.27)) hide)
     )
@@
       (project "sdrac_board"
         (path "/7e6d1db5-12f1-49d6-b3bd-d624ec5345e8/0c32a19a-a7ea-4fd5-9033-ebbe7320ca24"
-          (reference "#PWR095") (unit 1)
+          (reference "#PWR0101") (unit 1)
         )
       )
@@
   (symbol (lib_id "Device:R") (at 82.55 73.66 0) (unit 1)
     (in_bom yes) (on_board yes) (dnp no)
-    (property "Reference" "R41" (at 83.82 72.39 0)
+    (property "Reference" "R47" (at 83.82 72.39 0)
       (effects (font (size 1.27 1.27)) (justify left))
     )
@@
       (project "sdrac_board"
         (path "/7e6d1db5-12f1-49d6-b3bd-d624ec5345e8/0c32a19a-a7ea-4fd5-9033-ebbe7320ca24"
-          (reference "R41") (unit 1)
-        )
-      )
-      (project "motor controller"
-        (path "/98359aeb-e3f0-4579-a083-8ca5fb10d8d7/9635538f-af81-4033-8ebc-706153c1fd5e"
           (reference "R47") (unit 1)
         )
       )
+      (project "motor controller"
+        (path "/98359aeb-e3f0-4579-a083-8ca5fb10d8d7/9635538f-af81-4033-8ebc-706153c1fd5e"
+          (reference "R47") (unit 1)
+        )
+      )
     )
   )
   (symbol (lib_id "Device:R") (at 137.16 87.63 0) (unit 1)
     (in_bom yes) (on_board yes) (dnp no)
-    (property "Reference" "R42" (at 138.43 86.36 0)
+    (property "Reference" "R48" (at 138.43 86.36 0)
       (effects (font (size 1.27 1.27)) (justify left))
     )
@@
       (project "sdrac_board"
         (path "/7e6d1db5-12f1-49d6-b3bd-d624ec5345e8/0c32a19a-a7ea-4fd5-9033-ebbe7320ca24"
-          (reference "R42") (unit 1)
+          (reference "R48") (unit 1)
         )
       )
@@
   (symbol (lib_id "power:+3V3") (at 125.73 71.12 0) (unit 1)
     (in_bom yes) (on_board yes) (dnp no)
-    (property "Reference" "#PWR088" (at 125.73 74.93 0)
+    (property "Reference" "#PWR094" (at 125.73 74.93 0)
       (effects (font (size 1.27 1.27)) hide)
     )
@@
       (project "sdrac_board"
         (path "/7e6d1db5-12f1-49d6-b3bd-d624ec5345e8/0c32a19a-a7ea-4fd5-9033-ebbe7320ca24"
-          (reference "#PWR088") (unit 1)
+          (reference "#PWR094") (unit 1)
         )
       )
@@
   (symbol (lib_id "power:GND") (at 184.15 81.28 270) (unit 1)
     (in_bom yes) (on_board yes) (dnp no)
-    (property "Reference" "#PWR092" (at 177.8 81.28 0)
+    (property "Reference" "#PWR098" (at 177.8 81.28 0)
       (effects (font (size 1.27 1.27)) hide)
     )
@@
       (project "sdrac_board"
         (path "/7e6d1db5-12f1-49d6-b3bd-d624ec5345e8/0c32a19a-a7ea-4fd5-9033-ebbe7320ca24"
-          (reference "#PWR092") (unit 1)
+          (reference "#PWR098") (unit 1)
         )
       )
@@
   (symbol (lib_id "Device:R") (at 82.55 99.06 0) (unit 1)
     (in_bom yes) (on_board yes) (dnp no)
-    (property "Reference" "R43" (at 83.82 97.79 0)
+    (property "Reference" "R49" (at 83.82 97.79 0)
       (effects (font (size 1.27 1.27)) (justify left))
     )
@@
       (project "sdrac_board"
         (path "/7e6d1db5-12f1-49d6-b3bd-d624ec5345e8/0c32a19a-a7ea-4fd5-9033-ebbe7320ca24"
-          (reference "R43") (unit 1)
+          (reference "R49") (unit 1)
         )
       )
@@
   (symbol (lib_id "power:+5V") (at 184.15 97.79 0) (unit 1)
     (in_bom yes) (on_board yes) (dnp no)
-    (property "Reference" "#PWR096" (at 184.15 101.6 0)
+    (property "Reference" "#PWR0102" (at 184.15 101.6 0)
       (effects (font (size 1.27 1.27)) hide)
     )
@@
       (project "sdrac_board"
         (path "/7e6d1db5-12f1-49d6-b3bd-d624ec5345e8/0c32a19a-a7ea-4fd5-9033-ebbe7320ca24"
-          (reference "#PWR096") (unit 1)
-        )
-      )
+          (reference "#PWR0102") (unit 1)
+        )
+      )

Commit message: added 10A screw terminal
Parts:
- renumbered C49 to C50, J9 to J10, J10 to J11, J11 to J12, J12 to J13
