File: sdrac_board/Power.kicad_sch (KiCad schematic)
At the start: 41 parts, among them IC2 LMR16030PDDA, J2 Conn_01x02_Male, J3 Conn_01x02_Female, U6 AZ1117-3.3

Commit message: added second I2C communscation lane for synchronization and added wyas to change mcirosteping with resistors
Parts:
- renumbered C34 to C15, C44 to C16, C19 to C17, C20 to C18, C23 to C19, C25 to C20, C27 to C21, C29 to C22, C48 to C23, C49 to C24, C17 to C25, C12 to C26, C13 to C27, C15 to C28, C16 to C29, C22 to C30, C24 to C31, C26 to C32, C28 to C33, C18 to C34, C21 to C35, D10 to D7, D7 to D8, D8 to D9, IC2 to IC1, J2 to J4, J3 to J5, L2 to L1, L1 to L2, R22 to R19, R19 to R20, R23 to R21, R20 to R22, R21 to R23, R15 to R26, R17 to R27, R18 to R28, R16 to R29

Commit message: added hardware address selector
Parts:
- D7: footprint Diode_SMD:D_SMC -> Diode_SMD:D_SMA
- renumbered R19 to R25, R20 to R26, R21 to R27, R22 to R28, R23 to R29, R24 to R30, R25 to R31, R26 to R32, R27 to R33, R28 to R34, R29 to R35

Commit message: added 10A screw terminal
Parts:
- added C34: 1n, Capacitor_SMD:C_0603_1608Metric, symbol Device:C
- added J4: STEPER DRIVER VCC, TerminalBlock_Phoenix:TerminalBlock_Phoenix_MKDS-1,5-2_1x02_P5.00mm_Horizontal, symbol Connector:Screw_Terminal_01x02
- R32: value 100k -> 43k
- R35: value 10k -> 1k
- renumbered C34 to C35, C35 to C36, J4 to J5, J5 to J6
Connections:
- net +5V: now also C34.1
- net GND: now also C34.2, J4.1 (Pin_1)
- net VCC: now also J4.2 (Pin_2)

Commit message: fixwed resistors values
Parts:
- R32: value 43k -> 430k
- R35: value 1k -> 10k
Changed lines of the file:
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@@
       (effects (font (size 1.27 1.27)) (justify left))
     )
-    (property "Value" "43k" (at 31.75 175.26 0)
+    (property "Value" "430k" (at 31.75 175.26 0)
       (effects (font (size 1.27 1.27)) (justify left))
     )
@@
       (effects (font (size 1.27 1.27)) (justify left))
     )
-    (property "Value" "1k" (at 31.75 185.42 0)
-      (effects (font (size 1.27 1.27)) (justify left))
-    )
+    (property "Value" "10k" (at 31.75 185.42 0)
+      (effects (font (size 1.27 1.27)) (justify left))
+    )
